Commit message: .

File: humanoidverse/data/robots/g1/g1_23dof_lock_wrist.urdf (robot description, URDF)
Before this commit: robot g1_29dof_rev_1_0, 39 links, 38 joints
Joints:
- joint right_shoulder_pitch_joint: origin xyz=0.0039563 -0.10021 0.24778 rpy=-0.27931 5.4949E-05 0.00019159 -> xyz=0.0039563 -0.10022 0.24778 rpy=-0.27931 5.4949E-05 0.00019159
