Commit message: .

File: humanoidverse/data/robots/g1/g1_23dof_lock_wrist_symm_wrong0.urdf (robot description, URDF)
Before this commit: robot g1_29dof_rev_1_0, 39 links, 38 joints
Links:
- link logo_link: mass 0.001 -> 0.00001
Joints:
- joint head_joint: origin xyz=0.0039635 0 -0.044 rpy=0 0 0 -> xyz=0.0 0 -0.044 rpy=0 0 0
- joint waist_roll_joint: origin xyz=-0.0039635 0 0.044 rpy=0 0 0 -> xyz=-0.0 0 0.044 rpy=0 0 0
